File: new/tablet.kicad_sch (KiCad schematic)
At the start: 45 parts, among them J1 FSMC/TOUCH-SPI, J2 USB_B_Micro, J3 SD/CARD, J4 FLASH/FONT, J5 Conn_02x03_Odd_Even, J6 Conn_01x02, J7 Conn_ARM_SWD_TagConnect_TC2030, Q1 DMG2301L, SW1 SW_SPST, U1 STM32F429Z_E-G_Tx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

Commit message: add led
Parts:
- added D3, D4: LED_Small, Resistor_SMD:R_0603_1608Metric, symbol Device:LED_Small
- added R13, R14: 2k, Resistor_SMD:R_0603_1608Metric, symbol Device:R_Small
Connections:
- net GND: now also R13.2, R14.2
- net at U1.34 (PA0): now also D3.2 (A)
- net at U1.35 (PA1): now also D4.2 (A)
- new net: D4.1 (K), R14.1
- new net: D3.1 (K), R13.1
Changed lines of the file:
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@@
+    (stroke (width 0) (type default))
+  )
+  (wire (pts (xy 154.94 82.55) (xy 157.48 82.55))
     (stroke (width 0) (type default))
   )
@@
     (stroke (width 0) (type default))
   )
+  (wire (pts (xy 139.7 82.55) (xy 142.24 82.55))
+    (stroke (width 0) (type default))
+  )
   (wire (pts (xy 347.98 132.08) (xy 360.68 132.08))
     (stroke (width 0) (type default))
@@
     (stroke (width 0) (type default))
   )
+  (wire (pts (xy 147.32 80.01) (xy 149.86 80.01))
+    (stroke (width 0) (type default))
+  )
+  (wire (pts (xy 154.94 80.01) (xy 157.48 80.01))
+    (stroke (width 0) (type default))
+  )
+  (wire (pts (xy 142.24 80.01) (xy 139.7 80.01))
+    (stroke (width 0) (type default))
+  )
   (wire (pts (xy 116.84 30.48) (xy 119.38 30.48))
     (stroke (width 0) (type default))
@@
   )
   (wire (pts (xy 83.82 57.15) (xy 83.82 62.23))
+    (stroke (width 0) (type default))
+  )
+  (wire (pts (xy 147.32 82.55) (xy 149.86 82.55))
     (stroke (width 0) (type default))
   )
@@
         (path "/868516f5-1ea3-47ae-b277-3f67998564bb"
           (reference "C15") (unit 1)
+        )
+      )
+    )
+  )
+  (symbol (lib_id "power:GND") (at 157.48 82.55 90) (unit 1)
+    (in_bom yes) (on_board yes) (dnp no) (fields_autoplaced)
+    (property "Reference" "#PWR032" (at 163.83 82.55 0)
+      (effects (font (size 1.27 1.27)) hide)
+    )
+    (property "Value" "GND" (at 161.29 82.55 90)
+      (effects (font (size 1.27 1.27)) (justify right))
+    )
+    (property "Footprint" "" (at 157.48 82.55 0)
+      (effects (font (size 1.27 1.27)) hide)
+    )
+    (property "Datasheet" "" (at 157.48 82.55 0)
+      (effects (font (size 1.27 1.27)) hide)
+    )
+    (pin "1")
+    (instances
+      (project "tablet"
+        (path "/868516f5-1ea3-47ae-b277-3f67998564bb"
+          (reference "#PWR032") (unit 1)
         )
       )
@@
     )
   )
+  (symbol (lib_id "Device:LED_Small") (at 144.78 82.55 180) (unit 1)
+    (in_bom yes) (on_board yes) (dnp no) (fields_autoplaced)
+    (property "Reference" "D4" (at 144.7165 76.2 0)
+      (effects (font (size 1.27 1.27)))
+    )
+    (property "Value" "LED_Small" (at 144.7165 78.74 0)
+      (effects (font (size 1.27 1.27)))
+    )
+    (property "Footprint" "Resistor_SMD:R_0603_1608Metric" (at 144.78 82.55 90)
+      (effects (font (size 1.27 1.27)) hide)
+    )
+    (property "Datasheet" "~" (at 144.78 82.55 90)
+      (effects (font (size 1.27 1.27)) hide)
+    )
+    (pin "1")
+    (pin "2")
+    (instances
+      (project "tablet"
+        (path "/868516f5-1ea3-47ae-b277-3f67998564bb"
+          (reference "D4") (unit 1)
+        )
+      )
+    )
+  )
   (symbol (lib_id "power:GND") (at 203.2 125.73 180) (unit 1)
     (in_bom yes) (on_board yes) (dnp no) (fields_autoplaced)
@@
         (path "/868516f5-1ea3-47ae-b277-3f67998564bb"
           (reference "R6") (unit 1)
+        )
+      )
+    )
+  )
+  (symbol (lib_id "power:GND") (at 157.48 80.01 90) (unit 1)
+    (in_bom yes) (on_board yes) (dnp no) (fields_autoplaced)
+    (property "Reference" "#PWR031" (at 163.83 80.01 0)
+      (effects (font (size 1.27 1.27)) hide)
+    )
+    (property "Value" "GND" (at 161.29 80.01 90)
+      (effects (font (size 1.27 1.27)) (justify right))
+    )
+    (property "Footprint" "" (at 157.48 80.01 0)
+      (effects (font (size 1.27 1.27)) hide)
+    )
+    (property "Datasheet" "" (at 157.48 80.01 0)
+      (effects (font (size 1.27 1.27)) hide)
+    )
+    (pin "1")
+    (instances
+      (project "tablet"
+        (path "/868516f5-1ea3-47ae-b277-3f67998564bb"
+          (reference "#PWR031") (unit 1)
         )
       )
@@
     )
   )
+  (symbol (lib_id "Device:R_Small") (at 152.4 80.01 90) (unit 1)
+    (in_bom yes) (on_board yes) (dnp no) (fields_autoplaced)
+    (property "Reference" "R13" (at 152.4 74.93 90)
+      (effects (font (size 1.27 1.27)))
+    )
+    (property "Value" "2k" (at 152.4 77.47 90)
+      (effects (font (size 1.27 1.27)))
+    )
+    (property "Footprint" "Resistor_SMD:R_0603_1608Metric" (at 152.4 80.01 0)
+      (effects (font (size 1.27 1.27)) hide)
+    )
+    (property "Datasheet" "~" (at 152.4 80.01 0)
+      (effects (font (size 1.27 1.27)) hide)
+    )
+    (pin "1")
+    (pin "2")
+    (instances
+      (project "tablet"
+        (path "/868516f5-1ea3-47ae-b277-3f67998564bb"
+          (reference "R13") (unit 1)
+        )
+      )
+      (project "drone"
+        (path "/8d172cff-266e-4e68-aa3f-17546d01ba91"
+          (reference "R11") (unit 1)
+        )
+      )
+    )
+  )
   (symbol (lib_id "Diode:BAT48JFILM") (at 327.66 43.18 180) (unit 1)
     (in_bom yes) (on_board yes) (dnp no) (fields_autoplaced)
@@
         (path "/868516f5-1ea3-47ae-b277-3f67998564bb"
           (reference "D1") (unit 1)
+        )
+      )
+    )
+  )
+  (symbol (lib_id "Device:LED_Small") (at 144.78 80.01 180) (unit 1)
+    (in_bom yes) (on_board yes) (dnp no) (fields_autoplaced)
+    (property "Reference" "D3" (at 144.7165 73.66 0)
+      (effects (font (size 1.27 1.27)))
+    )
+    (property "Value" "LED_Small" (at 144.7165 76.2 0)
+      (effects (font (size 1.27 1.27)))
+    )
+    (property "Footprint" "Resistor_SMD:R_0603_1608Metric" (at 144.78 80.01 90)
+      (effects (font (size 1.27 1.27)) hide)
+    )
+    (property "Datasheet" "~" (at 144.78 80.01 90)
+      (effects (font (size 1.27 1.27)) hide)
+    )
+    (pin "1")
+    (pin "2")
+    (instances
+      (project "tablet"
+        (path "/868516f5-1ea3-47ae-b277-3f67998564bb"
+          (reference "D3") (unit 1)
         )
       )
@@
         )
       )
+    )
+  )
+  (symbol (lib_id "Device:R_Small") (at 152.4 82.55 90) (unit 1)
+    (in_bom yes) (on_board yes) (dnp no) (fields_autoplaced)
+    (property "Reference" "R14" (at 152.4 77.47 90)
+      (effects (font (size 1.27 1.27)))
+    )
+    (property "Value" "2k" (at 152.4 80.01 90)
+      (effects (font (size 1.27 1.27)))
+    )
+    (property "Footprint" "Resistor_SMD:R_0603_1608Metric" (at 152.4 82.55 0)
+      (effects (font (size 1.27 1.27)) hide)
+    )
+    (property "Datasheet" "~" (at 152.4 82.55 0)
+      (effects (font (size 1.27 1.27)) hide)
+    )
+    (pin "1")
+    (pin "2")
+    (instances
+      (project "tablet"
+        (path "/868516f5-1ea3-47ae-b277-3f67998564bb"
+          (reference "R14") (unit 1)
+        )
+      )
+      (project "drone"
+        (path "/8d172cff-266e-4e68-aa3f-17546d01ba91"
+          (reference "R11") (unit 1)
+        )
+      )
