File: new/tablet.kicad_pcb (KiCad board)
At the start: 2 copper layers, 132.7 x 75.8 mm, 45 parts, among them J1 FSMC/TOUCH-SPI, J2 USB_B_Micro, J3 SD/CARD, J4 FLASH/FONT, J5 Conn_02x03_Odd_Even, J6 Conn_01x02, J7 Conn_ARM_SWD_TagConnect_TC2030, Q1 DMG2301L, SW1 SW_SPST, U1 STM32F429Z_E-G_Tx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

Commit message: add led
Parts:
- added D3: LED_Small, Resistor_SMD:R_0603_1608Metric, F.Cu at (210.3, 149.4)
- added D4: LED_Small, Resistor_SMD:R_0603_1608Metric, F.Cu at (205.5, 149.4)
- added R13: 2k, Resistor_SMD:R_0603_1608Metric, F.Cu at (213.1, 149.4)
- added R14: 2k, Resistor_SMD:R_0603_1608Metric, F.Cu at (207.5, 149.4)
Connections:
- U1 pad 34: unconnected-(U1-PA0-Pad34) -> Net-(D3-A)
- U1 pad 35: unconnected-(U1-PA1-Pad35) -> Net-(D4-A)
Routing:
- net Net-(D3-A): track 0.00 -> 64.2 mm, vias 0 -> 2
- net Net-(D4-A): track 0.00 -> 62.4 mm, vias 0 -> 2
- net Net-(D3-K): track 0.00 -> 2.79 mm
- net Net-(D4-K): track 0.00 -> 2.03 mm
- net GND: vias 29 -> 30

Commit message: send for production
Connections:
- U1 pad 86: unconnected-(U1-PD15-Pad86) -> PD15-D1
Routing:
- net PD15-D1: track 0.00 -> 48.2 mm, vias 0 -> 2
- net PA14-SWCLK: track 39.4 -> 37.0 mm
- net PD1-D3: track 29.6 -> 30.7 mm
- net PD0-D2: track 24.3 -> 25.2 mm
